Commit message: add min logic to robotic node

File: workspaces/catkin_ws/src/launcher_robots_lab_robotica/urdf/ur3e_rg2_205_prefix.urdf (robot description, URDF)
Before this commit: robot ur3e_robot, 17 links, 16 joints
Links:
- removed link 205_base
- removed link 205_base_link
- removed link 205_base_link_inertia
- removed link 205_forearm_link
- removed link 205_left_inner_finger
- removed link 205_left_inner_knuckle
- removed link 205_left_outer_knuckle
- removed link 205_onrobot_rg2_base_link
- removed link 205_right_inner_finger
- removed link 205_right_inner_knuckle
- removed link 205_right_outer_knuckle
- removed link 205_shoulder_link
- removed link 205_tool0
- removed link 205_upper_arm_link
- removed link 205_wrist_1_link
- removed link 205_wrist_2_link
- removed link 205_wrist_3_link
- added link base_205
- added link base_link
- added link base_link_inertia_205, mass 2.0; collision mesh filename=package://launcher_robots_lab_robotica/meshes/collision/bas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; visual mesh filename=package://launcher_robots_lab_robotica/meshes/visual/base.d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
- added link forearm_link_205, mass 1.26; collision mesh filename=package://launcher_robots_lab_robotica/meshes/collision/for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; visual mesh filename=package://launcher_robots_lab_robotica/meshes/visual/forear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
- added link left_inner_finger_205, mass 0.05; collision mesh filename=package://launcher_robots_lab_robotica/meshes/collision/inn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; visual mesh filename=package://launcher_robots_lab_robotica/meshes/visual/inner_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
- added link left_inner_knuckle_205, mass 0.05; collision mesh filename=package://launcher_robots_lab_robotica/meshes/collision/inn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; visual mesh filename=package://launcher_robots_lab_robotica/meshes/visual/inner_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
- added link left_outer_knuckle_205, mass 0.05; collision mesh filename=package://launcher_robots_lab_robotica/meshes/collision/out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; visual mesh filename=package://launcher_robots_lab_robotica/meshes/visual/outer_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
- added link onrobot_rg2_base_link_205, mass 0.7; collision mesh filename=package://launcher_robots_lab_robotica/meshes/collision/bas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; visual mesh filename=package://launcher_robots_lab_robotica/meshes/visual/base_l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
- added link right_inner_finger_205, mass 0.05; collision mesh filename=package://launcher_robots_lab_robotica/meshes/collision/inn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; visual mesh filename=package://launcher_robots_lab_robotica/meshes/visual/inner_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
- added link right_inner_knuckle_205, mass 0.05; collision mesh filename=package://launcher_robots_lab_robotica/meshes/collision/inn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; visual mesh filename=package://launcher_robots_lab_robotica/meshes/visual/inner_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
- added link right_outer_knuckle_205, mass 0.05; collision mesh filename=package://launcher_robots_lab_robotica/meshes/collision/out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; visual mesh filename=package://launcher_robots_lab_robotica/meshes/visual/outer_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
- added link shoulder_link_205, mass 2.0; collision mesh filename=package://launcher_robots_lab_robotica/meshes/collision/sho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; visual mesh filename=package://launcher_robots_lab_robotica/meshes/visual/should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
- added link tool0_205
- added link upper_arm_link_205, mass 3.42; collision mesh filename=package://launcher_robots_lab_robotica/meshes/collision/upp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; visual mesh filename=package://launcher_robots_lab_robotica/meshes/visual/uppera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
- added link wrist_1_link_205, mass 0.8; collision mesh filename=package://launcher_robots_lab_robotica/meshes/collision/wri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; visual mesh filename=package://launcher_robots_lab_robotica/meshes/visual/wrist1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
- added link wrist_2_link_205, mass 0.8; collision mesh filename=package://launcher_robots_lab_robotica/meshes/collision/wri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; visual mesh filename=package://launcher_robots_lab_robotica/meshes/visual/wrist2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
- added link wrist_3_link_205, mass 0.35; collision mesh filename=package://launcher_robots_lab_robotica/meshes/collision/wri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; visual mesh filename=package://launcher_robots_lab_robotica/meshes/visual/wrist3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
Joints:
- removed joint 205_base_link-base_fixed_joint
- removed joint 205_base_link-base_link_inertia
- removed joint 205_elbow_joint
- removed joint 205_finger_joint
- removed joint 205_joint0
- removed joint 205_left_inner_finger_joint
- removed joint 205_left_inner_knuckle_joint
- removed joint 205_right_inner_finger_joint
- removed joint 205_right_inner_knuckle_joint
- removed joint 205_right_outer_knuckle_joint
- removed joint 205_shoulder_lift_joint
- removed joint 205_shoulder_pan_joint
- removed joint 205_wrist_1_joint
- removed joint 205_wrist_2_joint
- removed joint 205_wrist_3-tool0
- removed joint 205_wrist_3_joint
- added joint base_link-base_fixed_joint_205: type fixed, parent base_link, child base_205, origin xyz=0 0 0 rpy=0 0 3.141592653589793
- added joint base_link-base_link_inertia_205: type fixed, parent base_link, child base_link_inertia_205, origin xyz=0 0 0 rpy=0 0 3.141592653589793
- added joint elbow_joint_205: type revolute, parent upper_arm_link_205, child forearm_link_205, origin xyz=-0.2436650957547605 0 0 rpy=3.141429134391114 3.1413007534876 3.141585104530758, axis 0 0 1, limit lower=-3.141592653589793 upper=3.141592653589793 effort=28.0 velocity=3.141592653589793
- added joint finger_joint_205: type revolute, parent onrobot_rg2_base_link_205, child left_outer_knuckle_205, origin xyz=0 -0.017178 0.125797 rpy=0 0 0, axis -1 0 0, limit lower=-0.558505 upper=0.785398 effort=1000 velocity=100.0
- added joint joint0_205: type fixed, parent tool0_205, child onrobot_rg2_base_link_205, origin xyz=0. 0. 0. rpy=0.0 1.5707963267948966 0.0
- added joint left_inner_finger_joint_205: type revolute, parent left_outer_knuckle_205, child left_inner_finger_205, origin xyz=0 -0.039592 0.038177000000000016 rpy=0 0 0, axis 1 0 0, limit lower=-0.872665 upper=0.872665 effort=1000 velocity=100.0, mimic joint=finger_joint_205 multiplier=1 offset=0
- added joint left_inner_knuckle_joint_205: type revolute, parent onrobot_rg2_base_link_205, child left_inner_knuckle_205, origin xyz=0 -0.007678 0.1422970 rpy=0 0 0.0, axis 1 0 0, limit lower=-0.785398 upper=0.785398 effort=1000 velocity=100.0, mimic joint=finger_joint_205 multiplier=-1 offset=0
- added joint right_inner_finger_joint_205: type revolute, parent right_outer_knuckle_205, child right_inner_finger_205, origin xyz=0 -0.039592 0.038177000000000016 rpy=0 0 0, axis 1 0 0, limit lower=-0.872665 upper=0.872665 effort=1000 velocity=100.0, mimic joint=finger_joint_205 multiplier=1 offset=0
- added joint right_inner_knuckle_joint_205: type revolute, parent onrobot_rg2_base_link_205, child right_inner_knuckle_205, origin xyz=0 0.007678 0.1422970 rpy=0 0 -3.141592653589793, axis 1 0 0, limit lower=-0.785398 upper=0.785398 effort=1000 velocity=100.0, mimic joint=finger_joint_205 multiplier=-1 offset=0
- added joint right_outer_knuckle_joint_205: type revolute, parent onrobot_rg2_base_link_205, child right_outer_knuckle_205, origin xyz=0 0.017178 0.125797 rpy=0 0 3.141592653589793, axis 1 0 0, limit lower=-0.785398 upper=0.785398 effort=1000 velocity=100.0, mimic joint=finger_joint_205 multiplier=-1 offset=0
- added joint shoulder_lift_joint_205: type revolute, parent shoulder_link_205, child upper_arm_link_205, origin xyz=-0.000133574490397829 0 0 rpy=1.571184054925294 0 3.46931133972767e-07, axis 0 0 1, limit lower=-6.283185307179586 upper=6.283185307179586 effort=56.0 velocity=3.141592653589793
- added joint shoulder_pan_joint_205: type revolute, parent base_link_inertia_205, child shoulder_link_205, origin xyz=0 0 0.1519932046329507 rpy=0 0 -1.218598534562937e-07, axis 0 0 1, limit lower=-6.283185307179586 upper=6.283185307179586 effort=56.0 velocity=3.141592653589793
- added joint wrist_1_joint_205: type revolute, parent forearm_link_205, child wrist_1_link_205, origin xyz=-0.2131937361714605 -0.0007020488731425266 0.1309164554311118 rpy=0.00536252025231981 0.0008389012176466991 6.286415122585481e-06, axis 0 0 1, limit lower=-6.283185307179586 upper=6.283185307179586 effort=12.0 velocity=6.283185307179586
- added joint wrist_2_joint_205: type revolute, parent wrist_1_link_205, child wrist_2_link_205, origin xyz=8.773921560453022e-06 -0.08546373128392754 -7.049413943712751e-05 rpy=1.571621169361338 0 -1.170707376603464e-06, axis 0 0 1, limit lower=-6.283185307179586 upper=6.283185307179586 effort=12.0 velocity=6.283185307179586
- added joint wrist_3-tool0_205: type fixed, parent wrist_3_link_205, child tool0_205, origin xyz=0 0 0 rpy=0 -1.5707963267948966 -1.5707963267948966
- added joint wrist_3_joint_205: type revolute, parent wrist_2_link_205, child wrist_3_link_205, origin xyz=-0.0001118912945880604 0.09206143807114163 -0.0001405802282309842 rpy=1.569269301778692 3.141592653589793 -3.141592499182456, axis 0 0 1, limit lower=-6.283185307179586 upper=6.283185307179586 effort=12.0 velocity=6.283185307179586

File: workspaces/catkin_ws/src/launcher_robots_lab_robotica/urdf/ur3e_rg2_206_prefix.urdf (robot description, URDF)
Before this commit: robot ur3e_robot, 17 links, 16 joints
Links:
- removed link 206_base
- removed link 206_base_link
- removed link 206_base_link_inertia
- removed link 206_forearm_link
- removed link 206_left_inner_finger
- removed link 206_left_inner_knuckle
- removed link 206_left_outer_knuckle
- removed link 206_onrobot_rg2_base_link
- removed link 206_right_inner_finger
- removed link 206_right_inner_knuckle
- removed link 206_right_outer_knuckle
- removed link 206_shoulder_link
- removed link 206_tool0
- removed link 206_upper_arm_link
- removed link 206_wrist_1_link
- removed link 206_wrist_2_link
- removed link 206_wrist_3_link
- added link base_206
- added link base_link
- added link base_link_inertia_206, mass 2.0; collision mesh filename=package://launcher_robots_lab_robotica/meshes/collision/bas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; visual mesh filename=package://launcher_robots_lab_robotica/meshes/visual/base.d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
- added link forearm_link_206, mass 1.26; collision mesh filename=package://launcher_robots_lab_robotica/meshes/collision/for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; visual mesh filename=package://launcher_robots_lab_robotica/meshes/visual/forear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
- added link left_inner_finger_206, mass 0.05; collision mesh filename=package://launcher_robots_lab_robotica/meshes/collision/inn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; visual mesh filename=package://launcher_robots_lab_robotica/meshes/visual/inner_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
- added link left_inner_knuckle_206, mass 0.05; collision mesh filename=package://launcher_robots_lab_robotica/meshes/collision/inn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; visual mesh filename=package://launcher_robots_lab_robotica/meshes/visual/inner_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
- added link left_outer_knuckle_206, mass 0.05; collision mesh filename=package://launcher_robots_lab_robotica/meshes/collision/out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; visual mesh filename=package://launcher_robots_lab_robotica/meshes/visual/outer_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
- added link onrobot_rg2_base_link_206, mass 0.7; collision mesh filename=package://launcher_robots_lab_robotica/meshes/collision/bas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; visual mesh filename=package://launcher_robots_lab_robotica/meshes/visual/base_l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
- added link right_inner_finger_206, mass 0.05; collision mesh filename=package://launcher_robots_lab_robotica/meshes/collision/inn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; visual mesh filename=package://launcher_robots_lab_robotica/meshes/visual/inner_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
- added link right_inner_knuckle_206, mass 0.05; collision mesh filename=package://launcher_robots_lab_robotica/meshes/collision/inn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; visual mesh filename=package://launcher_robots_lab_robotica/meshes/visual/inner_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
- added link right_outer_knuckle_206, mass 0.05; collision mesh filename=package://launcher_robots_lab_robotica/meshes/collision/out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; visual mesh filename=package://launcher_robots_lab_robotica/meshes/visual/outer_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
- added link shoulder_link_206, mass 2.0; collision mesh filename=package://launcher_robots_lab_robotica/meshes/collision/sho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; visual mesh filename=package://launcher_robots_lab_robotica/meshes/visual/should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
- added link tool0_206
- added link upper_arm_link_206, mass 3.42; collision mesh filename=package://launcher_robots_lab_robotica/meshes/collision/upp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; visual mesh filename=package://launcher_robots_lab_robotica/meshes/visual/uppera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
- added link wrist_1_link_206, mass 0.8; collision mesh filename=package://launcher_robots_lab_robotica/meshes/collision/wri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; visual mesh filename=package://launcher_robots_lab_robotica/meshes/visual/wrist1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
- added link wrist_2_link_206, mass 0.8; collision mesh filename=package://launcher_robots_lab_robotica/meshes/collision/wri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; visual mesh filename=package://launcher_robots_lab_robotica/meshes/visual/wrist2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
- added link wrist_3_link_206, mass 0.35; collision mesh filename=package://launcher_robots_lab_robotica/meshes/collision/wri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; visual mesh filename=package://launcher_robots_lab_robotica/meshes/visual/wrist3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
Joints:
- removed joint 206_base_link-base_fixed_joint
- removed joint 206_base_link-base_link_inertia
- removed joint 206_elbow_joint
- removed joint 206_finger_joint
- removed joint 206_joint0
- removed joint 206_left_inner_finger_joint
- removed joint 206_left_inner_knuckle_joint
- removed joint 206_right_inner_finger_joint
- removed joint 206_right_inner_knuckle_joint
- removed joint 206_right_outer_knuckle_joint
- removed joint 206_shoulder_lift_joint
- removed joint 206_shoulder_pan_joint
- removed joint 206_wrist_1_joint
- removed joint 206_wrist_2_joint
- removed joint 206_wrist_3-tool0
- removed joint 206_wrist_3_joint
- added joint base_link-base_fixed_joint_206: type fixed, parent base_link, child base_206, origin xyz=0 0 0 rpy=0 0 3.141592653589793
- added joint base_link-base_link_inertia_206: type fixed, parent base_link, child base_link_inertia_206, origin xyz=0 0 0 rpy=0 0 3.141592653589793
- added joint elbow_joint_206: type revolute, parent upper_arm_link_206, child forearm_link_206, origin xyz=-0.2437259737936491 0 0 rpy=0.001105848958660876 0.0006034712402559254 -4.507836367124921e-06, axis 0 0 1, limit lower=-3.141592653589793 upper=3.141592653589793 effort=28.0 velocity=3.141592653589793
- added joint finger_joint_206: type revolute, parent onrobot_rg2_base_link_206, child left_outer_knuckle_206, origin xyz=0 -0.017178 0.125797 rpy=0 0 0, axis -1 0 0, limit lower=-0.558505 upper=0.785398 effort=1000 velocity=100.0
- added joint joint0_206: type fixed, parent tool0_206, child onrobot_rg2_base_link_206, origin xyz=0. 0. 0. rpy=0.0 1.5707963267948966 0.0
- added joint left_inner_finger_joint_206: type revolute, parent left_outer_knuckle_206, child left_inner_finger_206, origin xyz=0 -0.039592 0.038177000000000016 rpy=0 0 0, axis 1 0 0, limit lower=-0.872665 upper=0.872665 effort=1000 velocity=100.0, mimic joint=finger_joint_206 multiplier=1 offset=0
- added joint left_inner_knuckle_joint_206: type revolute, parent onrobot_rg2_base_link_206, child left_inner_knuckle_206, origin xyz=0 -0.007678 0.1422970 rpy=0 0 0.0, axis 1 0 0, limit lower=-0.785398 upper=0.785398 effort=1000 velocity=100.0, mimic joint=finger_joint_206 multiplier=-1 offset=0
- added joint right_inner_finger_joint_206: type revolute, parent right_outer_knuckle_206, child right_inner_finger_206, origin xyz=0 -0.039592 0.038177000000000016 rpy=0 0 0, axis 1 0 0, limit lower=-0.872665 upper=0.872665 effort=1000 velocity=100.0, mimic joint=finger_joint_206 multiplier=1 offset=0
- added joint right_inner_knuckle_joint_206: type revolute, parent onrobot_rg2_base_link_206, child right_inner_knuckle_206, origin xyz=0 0.007678 0.1422970 rpy=0 0 -3.141592653589793, axis 1 0 0, limit lower=-0.785398 upper=0.785398 effort=1000 velocity=100.0, mimic joint=finger_joint_206 multiplier=-1 offset=0
- added joint right_outer_knuckle_joint_206: type revolute, parent onrobot_rg2_base_link_206, child right_outer_knuckle_206, origin xyz=0 0.017178 0.125797 rpy=0 0 3.141592653589793, axis 1 0 0, limit lower=-0.785398 upper=0.785398 effort=1000 velocity=100.0, mimic joint=finger_joint_206 multiplier=-1 offset=0
- added joint shoulder_lift_joint_206: type revolute, parent shoulder_link_206, child upper_arm_link_206, origin xyz=-0.0001107110555958654 0 0 rpy=1.570329613154402 0 3.417864421477842e-06, axis 0 0 1, limit lower=-6.283185307179586 upper=6.283185307179586 effort=56.0 velocity=3.141592653589793
- added joint shoulder_pan_joint_206: type revolute, parent base_link_inertia_206, child shoulder_link_206, origin xyz=0 0 0.1519047144003236 rpy=0 0 -9.530599491829224e-08, axis 0 0 1, limit lower=-6.283185307179586 upper=6.283185307179586 effort=56.0 velocity=3.141592653589793
- added joint wrist_1_joint_206: type revolute, parent forearm_link_206, child wrist_1_link_206, origin xyz=-0.2132584137315163 -0.0004232381093861393 0.1311440944208638 rpy=0.003227264192714675 0.0009285627531319139 7.543943465429524e-07, axis 0 0 1, limit lower=-6.283185307179586 upper=6.283185307179586 effort=12.0 velocity=6.283185307179586
- added joint wrist_2_joint_206: type revolute, parent wrist_1_link_206, child wrist_2_link_206, origin xyz=0.000165700073623267 -0.08547162011592442 -0.0001881112192972863 rpy=1.572997184989922 0 1.978861212743183e-06, axis 0 0 1, limit lower=-6.283185307179586 upper=6.283185307179586 effort=12.0 velocity=6.283185307179586
- added joint wrist_3-tool0_206: type fixed, parent wrist_3_link_206, child tool0_206, origin xyz=0 0 0 rpy=0 -1.5707963267948966 -1.5707963267948966
- added joint wrist_3_joint_206: type revolute, parent wrist_2_link_206, child wrist_3_link_206, origin xyz=-9.449984879160511e-05 0.0920975245267849 -9.62025620790864e-05 rpy=1.569751754450705 3.141592653589793 3.141592261980481, axis 0 0 1, limit lower=-6.283185307179586 upper=6.283185307179586 effort=12.0 velocity=6.283185307179586
